Commit message: second_commit

File: robots/hustac_pg_v3.urdf (robot description, URDF)
Before this commit: robot hustac_pg_v3, 27 links, 26 joints
Links:
- link right_ee_link: mass 0.00506893153791104 -> 0.00506893153791106
Joints:
- joint left_ee_joint: origin xyz=-0.011 0.0105 0.022181 rpy=1.5708 6.4022E-19 2.2426E-16 -> xyz=-0.0110000000000008 0.0105000000000003 0.0221811953944651 rpy=1.5707963267949 6.40215462385206E-19 2.24264473650599E-16
- joint left_ee_joint2: origin xyz=0.011 0.0105 0.022181 rpy=1.5708 6.4022E-19 2.2426E-16 -> xyz=0.0110000000000001 0.0105000000000002 0.0221811953944651 rpy=1.5707963267949 6.40215462385206E-19 2.24264473650599E-16
- joint left_joint1: origin xyz=0 0.222 0.61 rpy=-3.473E-17 5.9674E-16 -3.1416 -> xyz=0 0.222 0.61 rpy=-3.47304729036467E-17 5.96744875736022E-16 -3.14159265358979
- joint left_joint2: origin xyz=0 -0.085 0 rpy=1.7042 1.5708 0.13344 -> xyz=0 -0.0849999999999999 0 rpy=1.70423675438618 1.57079631189374 0.133440427591288
- joint left_joint3: origin xyz=0 -0.35 0 rpy=-1.5708 9.3445E-17 3.1416 -> xyz=0 -0.35 0 rpy=-1.5707963267949 9.34447673947081E-17 3.14159265358979
- joint left_joint4: origin xyz=0 -0.099 0 rpy=-1.5708 -1.1102E-16 -3.1416 -> xyz=0 -0.0990000000000001 0 rpy=-1.5707963267949 -1.11022302462516E-16 -3.14159265358979
- joint left_joint5: origin xyz=0 -0.3 0 rpy=-1.5708 -1.609E-16 3.1416 -> xyz=0 -0.3 0 rpy=-1.5707963267949 -1.60902701370267E-16 3.14159265358979
- joint left_joint6: origin xyz=0 -0.064 0 rpy=-1.5708 6.9389E-18 -3.1416 -> xyz=0 -0.0640000000000001 0 rpy=-1.5707963267949 6.93889390390723E-18 -3.14159265358979
- joint left_joint7: origin xyz=0 -0.034 0 rpy=1.5708 1.5708 0 -> xyz=0 -0.034 0 rpy=1.5707963267949 1.5707963267949 0
- joint right_ee_joint: origin xyz=0.011 -0.0105 0.022181 rpy=1.5708 7.4751E-18 -3.1416 -> xyz=0.0110000000000067 -0.0104999999999925 0.0221811953944649 rpy=1.5707963267949 7.47513322448154E-18 -3.14159265358979
- joint right_ee_joint2: origin xyz=-0.011 -0.0105 0.022181 rpy=1.5708 7.4751E-18 -3.1416 -> xyz=-0.0110000000000009 -0.0104999999999998 0.0221811953944632 rpy=1.5707963267949 7.47513322448154E-18 -3.14159265358979
- joint right_joint1: origin xyz=0 -0.222 0.57 rpy=7.1471E-16 -1.449E-16 -1.5708 -> xyz=0 -0.222 0.61 rpy=-1.44900829258215E-16 -7.14706072102445E-16 2.84494650060195E-15
- joint right_joint2: origin xyz=0.045 0 0.04 rpy=1.5708 3.4694E-16 1.5708 -> xyz=0 -0.085 0 rpy=1.5707963267949 -1.5707963267949 0
- joint right_joint3: origin xyz=0.045 0 0.04 rpy=0 -1.5708 0 -> xyz=0 -0.35 0 rpy=-1.5707963267949 4.69556343789277E-17 3.14159265358979
- joint right_joint4: origin xyz=0.045 0 0.305 rpy=0 -1.5708 0 -> xyz=0 -0.0990000000000004 0 rpy=-1.5707963267949 -6.93889390390723E-18 3.14159265358979
- joint right_joint5: origin xyz=0.035 0 0.054 rpy=0 -1.5708 0 -> xyz=0 -0.3 0 rpy=-1.5707963267949 1.38489731979257E-16 -3.14159265358979
- joint right_joint6: origin xyz=0.034 0 0.265 rpy=-2.1235 -1.5708 -1.0181 -> xyz=0 -0.0639999999999999 0 rpy=-1.5707963267949 -1.11022302462516E-16 -3.14159265358979
- joint right_joint7: origin xyz=0.034 0 0.03 rpy=1.4901E-08 1.5708 0 -> xyz=0 -0.034 0 rpy=1.5707963267949 1.5707963267949 0
